Commit message: new big update everythintg

File: src/kafeiche_description/urdf/kafeiche_base.xacro (robot description, xacro)
@@ -6,11 +6,9 @@
   name="kafeiche"
   xmlns:xacro="http://www.ros.org/wiki/xacro">
-    <!-- Matherials -->
+	<!-- Variables -->
+	<xacro:property name="clearance" value="0.15" />
+	<!-- Matherials -->
     <xacro:include filename="$(find kafeiche_description)/urdf/kafeiche_materials.xacro" />
     <!-- Wheels and bases for them -->
-    <xacro:property name="wheel_radius" value="0.075"/>
-    <xacro:property name="wheel_separation" value="0.273"/>
-    <xacro:property name="wheel_width" value="0.03"/>
-    <xacro:property name="clearance" value="0.15" />
     <xacro:include filename="$(find kafeiche_description)/urdf/kafeiche_front_wheel_base.xacro" />
     <xacro:include filename="$(find kafeiche_description)/urdf/kafeiche_front_wheel.xacro" />
@@ -19,4 +17,7 @@
     <xacro:include filename="$(find kafeiche_description)/urdf/kafeiche_right_wheel_base.xacro" />
     <xacro:include filename="$(find kafeiche_description)/urdf/kafeiche_right_wheel.xacro" />
+	<!-- Ros2 Control hardware interfaces -->
+	<xacro:include filename="kafeiche_control.xacro" />
+	<parameters>$(find kafeiche_drivers)/config/kafeiche_controllers.yaml</parameters>
   <link
     name="kafeiche_base">

Commit message: upd

File: src/kafeiche_description/urdf/kafeiche_base.xacro (robot description, xacro)
@@ -1,14 +1,8 @@
 <?xml version="1.0" encoding="utf-8"?>
-<!-- This URDF was automatically created by SolidWorks to URDF Exporter! Originally created by Stephen Brawner (brawner@gmail.com)
-     Commit Version: 1.6.0-4-g7f85cfe  Build Version: 1.6.7995.38578
-     For more information, please see http://wiki.ros.org/sw_urdf_exporter -->
 <robot
   name="kafeiche"
   xmlns:xacro="http://www.ros.org/wiki/xacro">
-	<!-- Variables -->
-	<xacro:property name="clearance" value="0.15" />
-	<!-- Matherials -->
+    <xacro:property name="clearance" value="0.15" />
     <xacro:include filename="$(find kafeiche_description)/urdf/kafeiche_materials.xacro" />
-    <!-- Wheels and bases for them -->
     <xacro:include filename="$(find kafeiche_description)/urdf/kafeiche_front_wheel_base.xacro" />
     <xacro:include filename="$(find kafeiche_description)/urdf/kafeiche_front_wheel.xacro" />
@@ -17,7 +11,6 @@
     <xacro:include filename="$(find kafeiche_description)/urdf/kafeiche_right_wheel_base.xacro" />
     <xacro:include filename="$(find kafeiche_description)/urdf/kafeiche_right_wheel.xacro" />
-	<!-- Ros2 Control hardware interfaces -->
-	<xacro:include filename="$(find kafeiche_description)/urdf/kafeiche_control.xacro" />
-	<!-- Link for yaml <parameters>$(find kafeiche_drivers)/config/kafeiche_controllers.yaml</parameters>-->
+    <xacro:include filename="$(find kafeiche_description)/urdf/kafeiche_control.xacro" />
+    <parameters>$(find kafeiche_drivers)/config/kafeiche_controllers.yaml</parameters>
   <link
     name="kafeiche_base">

File: src/kafeiche_description/urdf/kafeiche_control.xacro (robot description, xacro)
@@ -8,9 +8,7 @@
 			</hardware>
 			<joint name="left_wheel_joint">
-				<!-- Интерфейсы команд для управления скоростью колеса (то чем мы можем управлять)-->
 				<command_interface name="velocity" />
-				  <param name="min">-5.1</param>
-				  <param name="max">5.1</param>
-				<!-- Интерфейсы состояния для чтения скорости с энкодера (то что мы можем только считывать) -->
+				  <param name="min">-10</param>
+				  <param name="max">10</param>
 				<state_interface name="position"/>
 				<state_interface name="velocity" />
@@ -18,6 +16,6 @@
 			<joint name="right_wheel_joint">
 				<command_interface name="velocity" />
-				  <param name="min">-5.1</param>
-				  <param name="max">5.1</param>
+				  <param name="min">-10</param>
+				  <param name="max">10</param>
 				<state_interface name="position"/>
 				<state_interface name="velocity" />
