Commit message: first iteration_not tasted!

File: src/kafeiche_description/urdf/kafeiche_control.xacro (robot description, xacro)
@@ -1,9 +1,10 @@
 <?xml version="1.0" encoding="utf-8"?>
 <robot xmlns:xacro="http://www.ros.org/wiki/xacro">
-		<ros2_control name="diffriver_system" type="system">
+		<ros2_control name="tricylcedriver_system" type="system">
 			<hardware>
-				<plugin>kafeiche_drivers/DiffKfc</plugin>
+				<plugin>kafeiche_drivers/TricylceKfc</plugin>
 				<param name="left_wheel_name">left_wheel_joint</param>
 				<param name="right_wheel_name">right_wheel_joint</param>
+				<param name="front_wheel_name">front_wheel_joint</param>
 			</hardware>
 			<joint name="left_wheel_joint">
@@ -11,5 +12,4 @@
 				  <param name="min">-2.54</param>
 				  <param name="max">2.54</param>
-				<state_interface name="position"/>
 				<state_interface name="velocity" />
 			</joint>
@@ -18,6 +18,9 @@
 				  <param name="min">-2.54</param>
 				  <param name="max">2.54</param>
+				<state_interface name="velocity" />
+			</joint>
+			<joint name="front_wheel_joint">
+				<command_interface name="position" />
 				<state_interface name="position"/>
-				<state_interface name="velocity" />
 			</joint>
 	</ros2_control>

Commit message: pre-reales TODO: remove not used code

File: src/kafeiche_description/urdf/kafeiche_control.xacro (robot description, xacro)
@@ -1,26 +1,22 @@
 <?xml version="1.0" encoding="utf-8"?>
 <robot xmlns:xacro="http://www.ros.org/wiki/xacro">
-		<ros2_control name="tricylcedriver_system" type="system">
+		<ros2_control name="tricycledriver_system" type="system">
 			<hardware>
-				<plugin>kafeiche_drivers/TricylceKfc</plugin>
+				<plugin>kafeiche_drivers/TricycleKfc</plugin>
 				<param name="left_wheel_name">left_wheel_joint</param>
 				<param name="right_wheel_name">right_wheel_joint</param>
 				<param name="front_wheel_name">front_wheel_joint</param>
 			</hardware>
+			<joint name="front_wheel_joint">
+				<command_interface name="position" />
+				<state_interface name="position"/>
+			</joint>
 			<joint name="left_wheel_joint">
 				<command_interface name="velocity" />
-				  <param name="min">-2.54</param>
-				  <param name="max">2.54</param>
 				<state_interface name="velocity" />
 			</joint>
 			<joint name="right_wheel_joint">
 				<command_interface name="velocity" />
-				  <param name="min">-2.54</param>
-				  <param name="max">2.54</param>
 				<state_interface name="velocity" />
-			</joint>
-			<joint name="front_wheel_joint">
-				<command_interface name="position" />
-				<state_interface name="position"/>
 			</joint>
 	</ros2_control>
